File: Board/Board.sch (EAGLE design)
At the start: 94 parts, among them Q1 SP0503BAHTG

Commit message: updated relay orientation
Parts:
- added R24: 100, rcl:R-EU_R0603
Connections:
- new net N$43: R24.2, T1.B
- net N$42: now also R24.1; no longer T1.B
Changed lines of the file:
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@@
 <part name="T1" library="transistor" library_urn="urn:adsk.eagle:library:402" deviceset="*-NPN-" device="SOT23-BEC" package3d_urn="urn:adsk.eagle:package:29919/2" technology="BC817-16"/>
 <part name="P+11" library="supply1" library_urn="urn:adsk.eagle:library:371" deviceset="V+" device=""/>
+<part name="R24" library="rcl" library_urn="urn:adsk.eagle:library:334" deviceset="R-EU_" device="R0603" package3d_urn="urn:adsk.eagle:package:23555/2" value="100"/>
 </parts>
 <sheets>
@@
 <instance part="T1" gate="G$1" x="66.04" y="279.4"/>
 <instance part="P+11" gate="1" x="68.58" y="289.56"/>
+<instance part="R24" gate="G$1" x="58.42" y="279.4"/>
 </instances>
 <busses>
@@
 <net name="N$42" class="0">
 <segment>
+<pinref part="555" gate="A" pin="Q"/>
+<wire x1="45.72" y1="279.4" x2="45.72" y2="274.32" width="0.1524" layer="91"/>
+<pinref part="R24" gate="G$1" pin="1"/>
+<wire x1="45.72" y1="279.4" x2="53.34" y2="279.4" width="0.1524" layer="91"/>
+</segment>
+</net>
+<net name="N$43" class="0">
+<segment>
 <pinref part="T1" gate="G$1" pin="B"/>
-<pinref part="555" gate="A" pin="Q"/>
-<wire x1="63.5" y1="279.4" x2="45.72" y2="279.4" width="0.1524" layer="91"/>
-<wire x1="45.72" y1="279.4" x2="45.72" y2="274.32" width="0.1524" layer="91"/>
-</segment>
-</net>
+<pinref part="R24" gate="G$1" pin="2"/>
+</segment>
+</net>
